File: apricot-kbd-uno.kicad_sch (KiCad schematic)
At the start: 8 parts, among them J101 Apricot Keyboard Port, U101 TSR_1-2450, U102 MC1488, U103 MC1489

Commit message: assembly documentation. rev. uno-1.0
Parts:
- removed D101: D, symbol Device:D
- A101: value Arduino_UNO_R3 -> (none); footprint Module:Arduino_UNO_R3 -> (none); now left out of the parts list
- C101: value C_Polarized_Small -> (none); now left out of the parts list
- U101: value TSR_1-2450 -> (none); footprint Converter_DCDC:Converter_DCDC_TRACO_TSR-1_THT -> (none)
- U102: value MC1488 -> (none); footprint Package_DIP:DIP-14_W7.62mm -> (none)
- U103: value MC1489 -> (none); footprint Package_DIP:DIP-14_W7.62mm -> (none)
Connections:
- net -12V: now also J101.4; no longer J101.7
- net Earth: now also A101.29 (GND), A101.6 (GND), A101.7 (GND), C101.2, J101.2, J101.7, J102.3, U101.2 (GND), U102.7 (GND), U103.7 (GND)
- net RS232.OUT: now also J101.5; no longer J101.2
- removed net GND: A101.29 (GND), A101.6 (GND), A101.7 (GND), C101.2, J101.8, J102.3, U101.2 (GND), U102.7 (GND), U103.7 (GND)
- no-connect marks 39 -> 38
Other:
- title: (none) -> PS/2 to Apricot Xi keyboard translator  
- moved on the sheet: A101, C101, J101, J102, U101, U102, U103
